File: MB.kicad_pcb (KiCad board)
At the start: 4 copper layers, 90.2 x 94.1 mm, 52 parts, among them J100 VCC INPUT, J101 SWITCH ON/OFF, J103 FAN VOLTAGE, J200 DOOR_OUTPUT, J300 MCP_EXTERNAL, J301 CAN_INPUT, K200 HF49FD/005-1H12T, Q100 WST4045, Q200 MMBT3904, U100 LM2596S-5, U101 AMS1117-3.3, U200 MEGA_PRO_EMBED_CH340G_{slash}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, U300 MCP2515-xSO, U301 TJA1051T-3, Y300 8MHz

Commit message: version validada
Parts:
- J101: footprint Connector_PinHeader_2.54mm:PinHeader_1x02_P2.54mm_Vertical -> B2B-XH-A:JST_B2B-XH-A_LF__SN_
- moved TP104 4.17 mm to (131.4, 52.4)
- moved TP100 2.44 mm to (131.4, 46.6)
- moved J101 1.21 mm to (132.1, 37.5), turned to 90 degrees
- moved H200 0.44 mm to (204.1, 44.1)
Routing:
- net /POWER/V_INPUT: track 27.0 -> 29.1 mm
- net GND: track 41.7 -> 42.6 mm, vias 346 -> 344
- net Net-(J101-Pin_2): track 11.5 -> 10.7 mm
Other:
- board text removed: "ATMEGA PRO 2560"
